Commit message: add wheel separately

File: m_hubo_omniWH_vrep.urdf (robot description, URDF)
Before this commit: robot m_hubo_omniWH, 38 links, 37 joints
Links:
- added link omniWH1, mass 0.480; collision mesh filename=/home/rainbow/catkin_ws/src/m_hubo/meshes/omni_wheel_col.STL; visual mesh filename=/home/rainbow/catkin_ws/src/m_hubo/meshes/omni_wheel.STL
- added link omniWH2, mass 0.480; collision mesh filename=/home/rainbow/catkin_ws/src/m_hubo/meshes/omni_wheel_col.STL; visual mesh filename=/home/rainbow/catkin_ws/src/m_hubo/meshes/omni_wheel.STL
- added link omniWH3, mass 0.480; collision mesh filename=/home/rainbow/catkin_ws/src/m_hubo/meshes/omni_wheel_col.STL; visual mesh filename=/home/rainbow/catkin_ws/src/m_hubo/meshes/omni_wheel.STL
- link Body_WHBase_link: geometry collision mesh filename=/home/rainbow/catkin_ws/src/m_hubo/meshes/mobile_hubo_lower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; visual mesh filename=/home/rainbow/catkin_ws/src/m_hubo/meshes/mobile_hubo_lower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
- link Body_vision: geometry collision mesh filename=/home/rainbow/catkin_ws/src/m_hubo/meshes/ASM_VISION_col.STL; visual mesh filename=/home/rainbow/catkin_ws/src/m_hubo/meshes/ASM_VISION.STL
Joints:
- added joint whbase_to_omniWH1: type continuous, parent Body_WHBase_link, child omniWH1, origin xyz=0.158 -0.27366 -0.075 rpy=0 0 -2.61799333, axis 0 1 0, limit effort=100000 velocity=2.0
- added joint whbase_to_omniWH2: type continuous, parent Body_WHBase_link, child omniWH2, origin xyz=0.158 0.27366 -0.075 rpy=0 0 -0.52359867, axis 0 1 0, limit effort=100000 velocity=2.0
- added joint whbase_to_omniWH3: type continuous, parent Body_WHBase_link, child omniWH3, origin xyz=-0.316 0.0 -0.075 rpy=0 0 1.570796, axis 0 1 0, limit effort=100000 velocity=2.0
- joint WST: origin xyz=0 0 0.692 rpy=0 0 0 -> xyz=0 0 0.677 rpy=0 0 0
