Commit message: updated 2019/3/5

File: mobile_hubo_omniWH/hubo_plugin/urdf/plannar_move_m_hubo_omniWH.urdf (robot description, URDF)
Before this commit: robot m_hubo_omniWH, 45 links, 44 joints
Links:
- link Body_LEB: geometry collision mesh filename=package://hubo_plugin/meshes/Body_LEB_col.STL; visual mesh filename=package://hubo_plugin/meshes/Body_LEB.STL
- link Body_LF1: geometry collision mesh filename=package://hubo_plugin/meshes/Body_LF1_col.STL; visual mesh filename=package://hubo_plugin/meshes/Body_LF1.STL
- link Body_LF2_a1: geometry collision mesh filename=package://hubo_plugin/meshes/Body_LF2_a1_col.STL; visual mesh filename=package://hubo_plugin/meshes/Body_LF2_a1.STL
- link Body_LF2_a2: geometry collision mesh filename=package://hubo_plugin/meshes/Body_LF2_a3_col.STL; visual mesh filename=package://hubo_plugin/meshes/Body_LF2_a2.STL
- link Body_LF2_a3: geometry collision mesh filename=package://hubo_plugin/meshes/Body_RF2_a3_col.STL; visual mesh filename=package://hubo_plugin/meshes/Body_LF2_a3.STL
- link Body_LF2_b1: geometry collision mesh filename=package://hubo_plugin/meshes/Body_LF2_b1_col.STL; visual mesh filename=package://hubo_plugin/meshes/Body_LF2_b1.STL
- link Body_LF2_b2: geometry collision mesh filename=package://hubo_plugin/meshes/Body_LF2_b2_col.STL; visual mesh filename=package://hubo_plugin/meshes/Body_LF2_b2.STL
- link Body_LF2_b3: geometry collision mesh filename=package://hubo_plugin/meshes/Body_LF2_b3_col.STL; visual mesh filename=package://hubo_plugin/meshes/Body_LF2_b3.STL
- link Body_LF2_c1: geometry collision mesh filename=package://hubo_plugin/meshes/Body_LF2_c1_col.STL; visual mesh filename=package://hubo_plugin/meshes/Body_LF2_c1.STL
- link Body_LF2_c2: geometry collision mesh filename=package://hubo_plugin/meshes/Body_LF2_c2_col.STL; visual mesh filename=package://hubo_plugin/meshes/Body_LF2_c2.STL
- link Body_LF2_c3: geometry collision mesh filename=package://hubo_plugin/meshes/Body_LF2_c3_col.STL; visual mesh filename=package://hubo_plugin/meshes/Body_LF2_c3.STL
- link Body_LSP: geometry collision mesh filename=package://hubo_plugin/meshes/Body_LSP_col.STL; visual mesh filename=package://hubo_plugin/meshes/Body_LSP.STL
- link Body_LSR: geometry collision mesh filename=package://hubo_plugin/meshes/Body_LSR_col.STL; visual mesh filename=package://hubo_plugin/meshes/Body_LSR.STL
- link Body_LSY: geometry collision mesh filename=package://hubo_plugin/meshes/Body_LSY_col.STL; visual mesh filename=package://hubo_plugin/meshes/Body_LSY.STL
- link Body_LWFT: geometry collision mesh filename=package://hubo_plugin/meshes/Body_LWFT_col.STL; visual mesh filename=package://hubo_plugin/meshes/Body_LWFT.STL
- link Body_LWP: geometry collision mesh filename=package://hubo_plugin/meshes/Body_LWP_col.STL; visual mesh filename=package://hubo_plugin/meshes/Body_LWP.STL
- link Body_LWY: geometry collision mesh filename=package://hubo_plugin/meshes/Body_LWY_col.STL; visual mesh filename=package://hubo_plugin/meshes/Body_LWY.STL
- link Body_REB: geometry collision mesh filename=package://hubo_plugin/meshes/Body_REB_col.STL; visual mesh filename=package://hubo_plugin/meshes/Body_REB.STL
- link Body_RF1: geometry collision mesh filename=package://hubo_plugin/meshes/Body_RF1_col.STL; visual mesh filename=package://hubo_plugin/meshes/Body_RF1.STL
- link Body_RF2_a1: geometry collision mesh filename=package://hubo_plugin/meshes/Body_RF2_a1_col.STL; visual mesh filename=package://hubo_plugin/meshes/Body_RF2_a1.STL
- link Body_RF2_a2: geometry collision mesh filename=package://hubo_plugin/meshes/Body_RF2_a2_col.STL; visual mesh filename=package://hubo_plugin/meshes/Body_RF2_a2.STL
- link Body_RF2_a3: geometry collision mesh filename=package://hubo_plugin/meshes/Body_RF2_a3_col.STL; visual mesh filename=package://hubo_plugin/meshes/Body_RF2_a3.STL
- link Body_RF2_b1: geometry collision mesh filename=package://hubo_plugin/meshes/Body_RF2_b1_col.STL; visual mesh filename=package://hubo_plugin/meshes/Body_RF2_b1.STL
- link Body_RF2_b2: geometry collision mesh filename=package://hubo_plugin/meshes/Body_RF2_b2_col.STL; visual mesh filename=package://hubo_plugin/meshes/Body_RF2_b2.STL
- link Body_RF2_b3: geometry collision mesh filename=package://hubo_plugin/meshes/Body_RF2_b3_col.STL; visual mesh filename=package://hubo_plugin/meshes/Body_RF2_b3.STL
- link Body_RF2_c1: geometry collision mesh filename=package://hubo_plugin/meshes/Body_RF2_c1_col.STL; visual mesh filename=package://hubo_plugin/meshes/Body_RF2_c1.STL
- link Body_RF2_c2: geometry collision mesh filename=package://hubo_plugin/meshes/Body_RF2_c2_col.STL; visual mesh filename=package://hubo_plugin/meshes/Body_RF2_c2.STL
- link Body_RF2_c3: geometry collision mesh filename=package://hubo_plugin/meshes/Body_RF2_c3_col.STL; visual mesh filename=package://hubo_plugin/meshes/Body_RF2_c3.STL
- link Body_RSP: geometry collision mesh filename=package://hubo_plugin/meshes/Body_RSP_col.STL; visual mesh filename=package://hubo_plugin/meshes/Body_RSP.STL
- link Body_RSR: geometry collision mesh filename=package://hubo_plugin/meshes/Body_RSR_col.STL; visual mesh filename=package://hubo_plugin/meshes/Body_RSR.STL
- link Body_RSY: geometry collision mesh filename=package://hubo_plugin/meshes/Body_RSY_col.STL; visual mesh filename=package://hubo_plugin/meshes/Body_RSY.STL
- link Body_RWFT: geometry collision mesh filename=package://hubo_plugin/meshes/Body_RWFT_col.STL; visual mesh filename=package://hubo_plugin/meshes/Body_RWFT.STL
- link Body_RWP: geometry collision mesh filename=package://hubo_plugin/meshes/Body_RWP_col.STL; visual mesh filename=package://hubo_plugin/meshes/Body_RWP.STL
- link Body_RWY: geometry collision mesh filename=package://hubo_plugin/meshes/Body_RWY_col.STL; visual mesh filename=package://hubo_plugin/meshes/Body_RWY.STL
- link Body_TORSO: geometry collision mesh filename=package://hubo_plugin/meshes/Body_TORSO_col.STL; visual mesh filename=package://hubo_plugin/meshes/Body_TORSO.STL
- link Body_WHBase_link: geometry collision mesh filename=package://hubo_plugin/meshes/OmniWheelBase_col.STL; visual mesh filename=package://hubo_plugin/meshes/OmniWheelBase.STL
- link Body_vision: geometry collision mesh filename=package://hubo_plugin/meshes/ASM_VISION_col.STL; visual mesh filename=package://hubo_plugin/meshes/ASM_VISION.STL
